Commit message: create bullet vehicle wrapper

File: models/vehicle.urdf (robot description, URDF)
Before this commit: robot vehicle, 5 links, 4 joints
Links:
- added link beam_left, mass 200.0; collision box size=3.5 0.3 0.3; visual box size=3.5 0.3 0.3
- added link beam_right, mass 200.0; collision box size=3.5 0.3 0.3; visual box size=3.5 0.3 0.3
Joints:
- added joint body_to_beam_left: type fixed, parent body, child beam_left, origin xyz=-1.25 0.6 0.9
- added joint body_to_beam_right: type fixed, parent body, child beam_right, origin xyz=-1.25 -0.6 0.9
- joint body_to_wheel_rl: origin xyz=-4 1.05 -0.75 -> xyz=-1.75 0.4 -1.65; parent body -> beam_left
- joint body_to_wheel_rr: origin xyz=-4 -1.05 -0.75 -> xyz=-1.75 -0.4 -1.65; parent body -> beam_right

File: models/vehicle.urdf.xacro (robot description, xacro)
@@ -12,4 +12,10 @@
   <xacro:property name="wheel_f_clear" value="0.1"/>
   <xacro:property name="wheel_r_x" value="-4"/>
+  <!-- Beam properties -->
+  <xacro:property name="beam_mass" value="200.0"/>
+  <xacro:property name="beam_length" value="3.5"/>
+  <xacro:property name="beam_width" value="0.3"/>
+  <xacro:property name="beam_height" value="0.3"/>
+  <!-- Macros -->
   <xacro:macro name="inertia_box" params="mass lx ly lz">
     <inertia
@@ -32,4 +38,14 @@
     />
   </xacro:macro>
+  <xacro:macro name="material_tire">
+    <material name="tire">
+      <color rgba="0.2392 0.2157 0.1686 1"/>
+    </material>
+    <contact>
+      <!-- ground plane has friction value of 1, so use
+        friction value for tire-groundtype that is found online. -->
+      <lateral_friction value="0.8"/>
+    </contact>
+  </xacro:macro>
   <link name="body">
     <inertial>
@@ -41,5 +57,4 @@
         <box size="${body_length} ${body_width} ${body_height}"/>
       </geometry>
-      <material name="blue"/>
     </visual>
     <collision>
@@ -49,4 +64,36 @@
     </collision>
   </link>
+  <link name="beam_left">
+    <inertial>
+      <mass value="${beam_mass}"/>
+      <xacro:inertia_box mass="${beam_mass}" lx="${beam_length}" ly="${beam_width}" lz="${beam_height}"/>
+    </inertial>
+    <visual>
+      <geometry>
+        <box size="${beam_length} ${beam_width} ${beam_height}"/>
+      </geometry>
+    </visual>
+    <collision>
+      <geometry>
+        <box size="${beam_length} ${beam_width} ${beam_height}"/>
+      </geometry>
+    </collision>
+  </link>
+  <link name="beam_right">
+    <inertial>
+      <mass value="${beam_mass}"/>
+      <xacro:inertia_box mass="${beam_mass}" lx="${beam_length}" ly="${beam_width}" lz="${beam_height}"/>
+    </inertial>
+    <visual>
+      <geometry>
+        <box size="${beam_length} ${beam_width} ${beam_height}"/>
+      </geometry>
+    </visual>
+    <collision>
+      <geometry>
+        <box size="${beam_length} ${beam_width} ${beam_height}"/>
+      </geometry>
+    </collision>
+  </link>
   <link name="wheel_fl">
     <inertial>
@@ -66,4 +113,5 @@
       <origin xyz="0 0 0" rpy="-1.57 0 0"/>
     </collision>
+    <xacro:material_tire />
   </link>
   <link name="wheel_rl">
@@ -84,4 +132,5 @@
       <origin xyz="0 0 0" rpy="-1.57 0 0"/>
     </collision>
+    <xacro:material_tire />
   </link>
   <link name="wheel_rr">
@@ -102,4 +151,5 @@
       <origin xyz="0 0 0" rpy="1.57 0 0"/>
     </collision>
+    <xacro:material_tire />
   </link>
   <link name="wheel_fr">
@@ -120,5 +170,17 @@
       <origin xyz="0 0 0" rpy="1.57 0 0"/>
     </collision>
-  </link>
+    <xacro:material_tire />
+  </link>
+  <!-- Beam joints -->
+  <joint name="body_to_beam_left" type="fixed">
+    <parent link="body"/>
+    <child link="beam_left"/>
+    <origin xyz="${body_length/2 - beam_length/2} ${body_width/2 - beam_width/2} ${body_height/2 + beam_height/2}"/>
+  </joint>
+  <joint name="body_to_beam_right" type="fixed">
+    <parent link="body"/>
+    <child link="beam_right"/>
+    <origin xyz="${body_length/2 - beam_length/2} ${-body_width/2 + beam_width/2} ${body_height/2 + beam_height/2}"/>
+  </joint>
   <joint name="body_to_wheel_fl" type="continuous">
     <parent link="body"/>
@@ -128,13 +190,13 @@
   </joint>
   <joint name="body_to_wheel_rl" type="continuous">
-    <parent link="body"/>
+    <parent link="beam_left"/>
     <child link="wheel_rl"/>
-    <origin xyz="${wheel_r_x} ${body_width/2 + wheel_width/2 + wheel_f_clear} ${-body_height/2}"/>
+    <origin xyz="${-beam_length/2} ${wheel_width} ${-body_height - beam_height/2}"/>
     <axis xyz="0 1 0"/>
   </joint>
   <joint name="body_to_wheel_rr" type="continuous">
-    <parent link="body"/>
+    <parent link="beam_right"/>
     <child link="wheel_rr"/>
-    <origin xyz="${wheel_r_x} ${-body_width/2 - wheel_width/2 - wheel_f_clear} ${-body_height/2}"/>
+    <origin xyz="${-beam_length/2} ${-wheel_width} ${-body_height - beam_height/2}"/>
     <axis xyz="0 1 0"/>
   </joint>
