Commit message: add steering axis

File: ws/src/simulator/models/simple_car/model.urdf (robot description, URDF)
Before this commit: robot simple_car, 5 links, 4 joints
Links:
- removed link wheel_link_fl
- removed link wheel_link_fr
- removed link wheel_link_rl
- removed link wheel_link_rr
- added link wheel_fl_base, mass 20; visual box size=0.3 0.3 0.3
- added link wheel_fl_tire, mass 50; collision cylinder length=0.3 radius=0.5; visual cylinder length=0.3 radius=0.5
- added link wheel_fr_base, mass 20; visual box size=0.3 0.3 0.3
- added link wheel_fr_tire, mass 50; collision cylinder length=0.3 radius=0.5; visual cylinder length=0.3 radius=0.5
- added link wheel_rl_base, mass 20; visual box size=0.3 0.3 0.3
- added link wheel_rl_tire, mass 50; collision cylinder length=0.3 radius=0.5; visual cylinder length=0.3 radius=0.5
- added link wheel_rr_base, mass 20; visual box size=0.3 0.3 0.3
- added link wheel_rr_tire, mass 50; collision cylinder length=0.3 radius=0.5; visual cylinder length=0.3 radius=0.5
Joints:
- removed joint joint_base_link_to_wheel_link_fl
- removed joint joint_base_link_to_wheel_link_fr
- removed joint joint_base_link_to_wheel_link_rl
- removed joint joint_base_link_to_wheel_link_rr
- added joint joint_base_link_to_wheel_fl_base: type continuous, parent base_link, child wheel_fl_base, origin xyz=2 2 0 rpy=0 0 0, axis 0 0 1
- added joint joint_base_link_to_wheel_fr_base: type continuous, parent base_link, child wheel_fr_base, origin xyz=2 -2 0 rpy=0 0 0, axis 0 0 1
- added joint joint_base_link_to_wheel_rl_base: type continuous, parent base_link, child wheel_rl_base, origin xyz=-2 2 0 rpy=0 0 0, axis 0 0 1
- added joint joint_base_link_to_wheel_rr_base: type continuous, parent base_link, child wheel_rr_base, origin xyz=-2 -2 0 rpy=0 0 0, axis 0 0 1
- added joint joint_base_to_wheel_fl_tire: type continuous, parent wheel_fl_base, child wheel_fl_tire, origin xyz=0 0 -1 rpy=1.5707963267948966 0 0, axis 0 0 1
- added joint joint_base_to_wheel_fr_tire: type continuous, parent wheel_fr_base, child wheel_fr_tire, origin xyz=0 0 -1 rpy=1.5707963267948966 0 0, axis 0 0 1
- added joint joint_base_to_wheel_rl_tire: type continuous, parent wheel_rl_base, child wheel_rl_tire, origin xyz=0 0 -1 rpy=1.5707963267948966 0 0, axis 0 0 1
- added joint joint_base_to_wheel_rr_tire: type continuous, parent wheel_rr_base, child wheel_rr_tire, origin xyz=0 0 -1 rpy=1.5707963267948966 0 0, axis 0 0 1

File: ws/src/simulator/models/simple_car/model.urdf.xacro (robot description, xacro)
@@ -28,6 +28,20 @@
         </link>
     </xacro:macro>
-    <xacro:macro name="link_cylinder" params="name mass radius length">
-        <link name="${name}">
+    <xacro:macro name="wheel" params="name parent mass radius length xyz">
+        <link name="${name}_base">
+            <inertial>
+                <origin xyz="0 0 0" rpy="0 0 0"/>
+                <mass value="20"/>
+                <inertia ixx="1" ixy="0" ixz="0"
+                    iyy="1" iyz="0"
+                    izz="1"/>
+            </inertial>
+            <visual>
+                <geometry>
+                    <box size="0.3 0.3 0.3"/>
+                </geometry>
+            </visual>
+        </link>
+        <link name="${name}_tire">
             <inertial>
                 <origin xyz="0 0 0" rpy="0 0 0"/>
@@ -50,21 +64,31 @@
             </collision>
         </link>
+        <joint name="joint_${parent}_to_${name}_base" type="continuous">
+            <origin xyz="${xyz}" rpy="0 0 0"/>
+            <parent link="${parent}"/>
+            <child link="${name}_base"/>
+            <axis xyz="0 0 1"/>
+        </joint>
+        <joint name="joint_base_to_${name}_tire" type="continuous">
+            <origin xyz="0 0 -1" rpy="${pi/2} 0 0"/>
+            <parent link="${name}_base"/>
+            <child link="${name}_tire"/>
+            <axis xyz="0 0 1"/>
+        </joint>
+        <gazebo reference="${name}_base">
+            <material>Gazebo/Blue</material>
+        </gazebo>
+        <gazebo reference="${name}_tire">
+            <material>Gazebo/Orange</material>
+            <mu1>0.8</mu1>
+            <mu2>0.5</mu2>
+        </gazebo>
     </xacro:macro>
     <xacro:macro name="wheel_joint" params="parent child xyz">
-        <joint name="joint_${parent}_to_${child}" type="continuous">
-            <origin xyz="${xyz}" rpy="${pi/2} 0 0"/>
-            <parent link="${parent}"/>
-            <child link="${child}"/>
-            <axis xyz="0 0 1"/>
-        </joint>
     </xacro:macro>
     <xacro:link_box name="base_link" mass="${body_mass}" length="2" width="0.8" height="0.5"/>
-    <xacro:link_cylinder name="wheel_link_fl" mass="${wheel_mass}" radius="${wheel_radius}" length="${wheel_length}"/>
-    <xacro:link_cylinder name="wheel_link_rl" mass="${wheel_mass}" radius="${wheel_radius}" length="${wheel_length}"/>
-    <xacro:link_cylinder name="wheel_link_rr" mass="${wheel_mass}" radius="${wheel_radius}" length="${wheel_length}"/>
-    <xacro:link_cylinder name="wheel_link_fr" mass="${wheel_mass}" radius="${wheel_radius}" length="${wheel_length}"/>
-    <xacro:wheel_joint parent="base_link" child="wheel_link_fl" xyz="2 2 0"/>
-    <xacro:wheel_joint parent="base_link" child="wheel_link_rl" xyz="-2 2 0"/>
-    <xacro:wheel_joint parent="base_link" child="wheel_link_rr" xyz="-2 -2 0"/>
-    <xacro:wheel_joint parent="base_link" child="wheel_link_fr" xyz="2 -2 0"/>
+    <xacro:wheel name="wheel_fl" parent="base_link" mass="${wheel_mass}" radius="${wheel_radius}" length="${wheel_length}" xyz="2 2 0"/>
+    <xacro:wheel name="wheel_rl" parent="base_link" mass="${wheel_mass}" radius="${wheel_radius}" length="${wheel_length}" xyz="-2 2 0"/>
+    <xacro:wheel name="wheel_rr" parent="base_link" mass="${wheel_mass}" radius="${wheel_radius}" length="${wheel_length}" xyz="-2 -2 0"/>
+    <xacro:wheel name="wheel_fr" parent="base_link" mass="${wheel_mass}" radius="${wheel_radius}" length="${wheel_length}" xyz="2 -2 0"/>
 </robot>

Commit message: add drive command listener to gazebo_plugin

File: ws/src/simulator/models/simple_car/model.urdf (robot description, URDF)
Before this commit: robot simple_car, 9 links, 8 joints
Links:
- added link wheel_fl_steer, mass 1; visual box size=0.3 0.3 0.15
- added link wheel_fr_steer, mass 1; visual box size=0.3 0.3 0.15
- added link wheel_rl_steer, mass 1; visual box size=0.3 0.3 0.15
- added link wheel_rr_steer, mass 1; visual box size=0.3 0.3 0.15
- link wheel_fl_base: mass 20 -> 1; geometry visual box size=0.3 0.3 0.15
- link wheel_fr_base: mass 20 -> 1; geometry visual box size=0.3 0.3 0.15
- link wheel_rl_base: mass 20 -> 1; geometry visual box size=0.3 0.3 0.15
- link wheel_rr_base: mass 20 -> 1; geometry visual box size=0.3 0.3 0.15
Joints:
- removed joint joint_base_to_wheel_fl_tire
- removed joint joint_base_to_wheel_fr_tire
- removed joint joint_base_to_wheel_rl_tire
- removed joint joint_base_to_wheel_rr_tire
- added joint joint_wheel_fl_base_to_wheel_fl_steer: type continuous, parent wheel_fl_base, child wheel_fl_steer, origin xyz=0 0 0 rpy=0 0 0, axis 0 0 1
- added joint joint_wheel_fl_steer_to_wheel_fl_tire: type continuous, parent wheel_fl_steer, child wheel_fl_tire, origin xyz=0 0 -0.65 rpy=1.5707963267948966 0 0, axis 0 0 1
- added joint joint_wheel_fr_base_to_wheel_fr_steer: type continuous, parent wheel_fr_base, child wheel_fr_steer, origin xyz=0 0 0 rpy=0 0 0, axis 0 0 1
- added joint joint_wheel_fr_steer_to_wheel_fr_tire: type continuous, parent wheel_fr_steer, child wheel_fr_tire, origin xyz=0 0 -0.65 rpy=1.5707963267948966 0 0, axis 0 0 1
- added joint joint_wheel_rl_base_to_wheel_rl_steer: type continuous, parent wheel_rl_base, child wheel_rl_steer, origin xyz=0 0 0 rpy=0 0 0, axis 0 0 1
- added joint joint_wheel_rl_steer_to_wheel_rl_tire: type continuous, parent wheel_rl_steer, child wheel_rl_tire, origin xyz=0 0 -0.65 rpy=1.5707963267948966 0 0, axis 0 0 1
- added joint joint_wheel_rr_base_to_wheel_rr_steer: type continuous, parent wheel_rr_base, child wheel_rr_steer, origin xyz=0 0 0 rpy=0 0 0, axis 0 0 1
- added joint joint_wheel_rr_steer_to_wheel_rr_tire: type continuous, parent wheel_rr_steer, child wheel_rr_tire, origin xyz=0 0 -0.65 rpy=1.5707963267948966 0 0, axis 0 0 1
- joint joint_base_link_to_wheel_fl_base: type continuous -> fixed
- joint joint_base_link_to_wheel_fr_base: type continuous -> fixed
- joint joint_base_link_to_wheel_rl_base: type continuous -> fixed
- joint joint_base_link_to_wheel_rr_base: type continuous -> fixed

File: ws/src/simulator/models/simple_car/model.urdf.xacro (robot description, xacro)
@@ -32,5 +32,5 @@
             <inertial>
                 <origin xyz="0 0 0" rpy="0 0 0"/>
-                <mass value="20"/>
+                <mass value="1"/>
                 <inertia ixx="1" ixy="0" ixz="0"
                     iyy="1" iyz="0"
@@ -38,6 +38,21 @@
             </inertial>
             <visual>
+                <origin xyz="0 0 0.075" rpy="0 0 0"/>
                 <geometry>
-                    <box size="0.3 0.3 0.3"/>
+                    <box size="0.3 0.3 0.15"/>
+                </geometry>
+            </visual>
+        </link>
+        <link name="${name}_steer">
+            <inertial>
+                <mass value="1"/>
+                <inertia ixx="1" ixy="0" ixz="0"
+                    iyy="1" iyz="0"
+                    izz="1"/>
+            </inertial>
+            <visual>
+                <origin xyz="0 0 -0.075" rpy="0 0 0"/>
+                <geometry>
+                    <box size="0.3 0.3 0.15"/>
                 </geometry>
             </visual>
@@ -64,5 +79,5 @@
             </collision>
         </link>
-        <joint name="joint_${parent}_to_${name}_base" type="continuous">
+        <joint name="joint_${parent}_to_${name}_base" type="fixed">
             <origin xyz="${xyz}" rpy="0 0 0"/>
             <parent link="${parent}"/>
@@ -70,11 +85,26 @@
             <axis xyz="0 0 1"/>
         </joint>
-        <joint name="joint_base_to_${name}_tire" type="continuous">
-            <origin xyz="0 0 -1" rpy="${pi/2} 0 0"/>
+        <joint name="joint_${name}_base_to_${name}_steer" type="continuous">
+            <origin xyz="0 0 0" rpy="0 0 0"/>
             <parent link="${name}_base"/>
+            <child link="${name}_steer"/>
+            <axis xyz="0 0 1"/>
+        </joint>
+        <joint name="joint_${name}_steer_to_${name}_tire" type="continuous">
+            <origin xyz="0 0 ${-radius - 0.15}" rpy="${pi/2} 0 0"/>
+            <parent link="${name}_steer"/>
             <child link="${name}_tire"/>
             <axis xyz="0 0 1"/>
         </joint>
-        <gazebo reference="${name}_base">
+        <transmission name="${name}_steer_transmission">
+            <type>transmission_interface/SimpleTransmission</type>
+            <actuator name="$${name}_steer_motor">
+                <mechanicalReduction>1</mechanicalReduction>
+            </actuator>
+            <joint name="joint_${name}_base_to_${name}_steer">
+                <hardwareInterface>hardware_interface/PositionJointInterface</hardwareInterface>
+            </joint>
+        </transmission>
+        <gazebo reference="${name}_steer">
             <material>Gazebo/Blue</material>
         </gazebo>
@@ -92,3 +122,10 @@
     <xacro:wheel name="wheel_rr" parent="base_link" mass="${wheel_mass}" radius="${wheel_radius}" length="${wheel_length}" xyz="-2 -2 0"/>
     <xacro:wheel name="wheel_fr" parent="base_link" mass="${wheel_mass}" radius="${wheel_radius}" length="${wheel_length}" xyz="2 -2 0"/>
+    <gazebo>
+        <plugin name="simple_car" filename="libsimple_car.so">
+            <ros>
+                <namespace>/vehicle_namespace</namespace>
+            </ros>
+        </plugin>
+    </gazebo>
 </robot>

Commit message: add steering and drive torques topic

File: ws/src/simulator/models/simple_car/model.urdf (robot description, URDF)
Before this commit: robot simple_car, 13 links, 12 joints
Joints:
- joint joint_wheel_fl_steer_to_wheel_fl_tire: origin xyz=0 0 -0.65 rpy=1.5707963267948966 0 0 -> xyz=0 0 -0.65 rpy=-1.5707963267948966 0 0
- joint joint_wheel_fr_steer_to_wheel_fr_tire: origin xyz=0 0 -0.65 rpy=1.5707963267948966 0 0 -> xyz=0 0 -0.65 rpy=-1.5707963267948966 0 0
- joint joint_wheel_rl_steer_to_wheel_rl_tire: origin xyz=0 0 -0.65 rpy=1.5707963267948966 0 0 -> xyz=0 0 -0.65 rpy=-1.5707963267948966 0 0
- joint joint_wheel_rr_steer_to_wheel_rr_tire: origin xyz=0 0 -0.65 rpy=1.5707963267948966 0 0 -> xyz=0 0 -0.65 rpy=-1.5707963267948966 0 0

File: ws/src/simulator/models/simple_car/model.urdf.xacro (robot description, xacro)
@@ -92,5 +92,5 @@
         </joint>
         <joint name="joint_${name}_steer_to_${name}_tire" type="continuous">
-            <origin xyz="0 0 ${-radius - 0.15}" rpy="${pi/2} 0 0"/>
+            <origin xyz="0 0 ${-radius - 0.15}" rpy="${-pi/2} 0 0"/>
             <parent link="${name}_steer"/>
             <child link="${name}_tire"/>

Commit message: remove unwanted files

File: ws/src/simulator/models/simple_car/model.urdf (robot description, URDF)
Before this commit: robot simple_car, 13 links, 12 joints
Links:
- link base_link: mass 50 -> 1580; geometry collision box size=1 1 1; visual box size=1 1 1
- link wheel_fl_tire: mass 50 -> 200; geometry collision cylinder length=0.4 radius=0.505; visual cylinder length=0.4 radius=0.505
- link wheel_fr_tire: mass 50 -> 200; geometry collision cylinder length=0.4 radius=0.505; visual cylinder length=0.4 radius=0.505
- link wheel_rl_tire: mass 50 -> 200; geometry collision cylinder length=0.4 radius=0.505; visual cylinder length=0.4 radius=0.505
- link wheel_rr_tire: mass 50 -> 200; geometry collision cylinder length=0.4 radius=0.505; visual cylinder length=0.4 radius=0.505
Joints:
- joint joint_base_link_to_wheel_fl_base: origin xyz=2 2 0 rpy=0 0 0 -> xyz=0.2 1 0 rpy=0 0 0
- joint joint_base_link_to_wheel_fr_base: origin xyz=2 -2 0 rpy=0 0 0 -> xyz=0.2 -1 0 rpy=0 0 0
- joint joint_base_link_to_wheel_rl_base: origin xyz=-2 2 0 rpy=0 0 0 -> xyz=-3 1 0 rpy=0 0 0
- joint joint_base_link_to_wheel_rr_base: origin xyz=-2 -2 0 rpy=0 0 0 -> xyz=-3 -1 0 rpy=0 0 0
- joint joint_wheel_fl_steer_to_wheel_fl_tire: origin xyz=0 0 -0.65 rpy=-1.5707963267948966 0 0 -> xyz=0 0 -0.655 rpy=-1.5707963267948966 0 0
- joint joint_wheel_fr_steer_to_wheel_fr_tire: origin xyz=0 0 -0.65 rpy=-1.5707963267948966 0 0 -> xyz=0 0 -0.655 rpy=-1.5707963267948966 0 0
- joint joint_wheel_rl_steer_to_wheel_rl_tire: origin xyz=0 0 -0.65 rpy=-1.5707963267948966 0 0 -> xyz=0 0 -0.655 rpy=-1.5707963267948966 0 0
- joint joint_wheel_rr_steer_to_wheel_rr_tire: origin xyz=0 0 -0.65 rpy=-1.5707963267948966 0 0 -> xyz=0 0 -0.655 rpy=-1.5707963267948966 0 0

File: ws/src/simulator/models/simple_car/model.urdf.xacro (robot description, xacro)
@@ -1,8 +1,8 @@
 <?xml version="1.0"?>
 <robot xmlns:xacro="http://www.ros.org/wiki/xacro" name="simple_car">
-    <xacro:property name="wheel_mass" value="50"/>
-    <xacro:property name="wheel_radius" value="0.5"/>
-    <xacro:property name="wheel_length" value="0.3"/>
-    <xacro:property name="body_mass" value="50"/>
+    <xacro:property name="wheel_mass" value="200"/>
+    <xacro:property name="wheel_radius" value="0.505"/>
+    <xacro:property name="wheel_length" value="0.4"/>
+    <xacro:property name="body_mass" value="1580"/>
     <xacro:macro name="link_box" params="name mass length width height">
         <link name="${name}">
@@ -117,9 +117,9 @@
     <xacro:macro name="wheel_joint" params="parent child xyz">
     </xacro:macro>
-    <xacro:link_box name="base_link" mass="${body_mass}" length="2" width="0.8" height="0.5"/>
-    <xacro:wheel name="wheel_fl" parent="base_link" mass="${wheel_mass}" radius="${wheel_radius}" length="${wheel_length}" xyz="2 2 0"/>
-    <xacro:wheel name="wheel_rl" parent="base_link" mass="${wheel_mass}" radius="${wheel_radius}" length="${wheel_length}" xyz="-2 2 0"/>
-    <xacro:wheel name="wheel_rr" parent="base_link" mass="${wheel_mass}" radius="${wheel_radius}" length="${wheel_length}" xyz="-2 -2 0"/>
-    <xacro:wheel name="wheel_fr" parent="base_link" mass="${wheel_mass}" radius="${wheel_radius}" length="${wheel_length}" xyz="2 -2 0"/>
+    <xacro:link_box name="base_link" mass="${body_mass}" length="1" width="1" height="1"/>
+    <xacro:wheel name="wheel_fl" parent="base_link" mass="${wheel_mass}" radius="${wheel_radius}" length="${wheel_length}" xyz="0.2 1 0"/>
+    <xacro:wheel name="wheel_rl" parent="base_link" mass="${wheel_mass}" radius="${wheel_radius}" length="${wheel_length}" xyz="-3 1 0"/>
+    <xacro:wheel name="wheel_rr" parent="base_link" mass="${wheel_mass}" radius="${wheel_radius}" length="${wheel_length}" xyz="-3 -1 0"/>
+    <xacro:wheel name="wheel_fr" parent="base_link" mass="${wheel_mass}" radius="${wheel_radius}" length="${wheel_length}" xyz="0.2 -1 0"/>
     <gazebo>
         <plugin name="simple_car" filename="libsimple_car.so">
