Commit message: split gazebo plugin into two components

File: ws/src/simulator/models/simple_car/model.urdf.xacro (robot description, xacro)
@@ -28,5 +28,5 @@
         </link>
     </xacro:macro>
-    <xacro:macro name="wheel" params="name parent mass radius length xyz">
+    <xacro:macro name="wheel_macro" params="name parent mass radius length xyz">
         <link name="${name}_base">
             <inertial>
@@ -97,13 +97,15 @@
             <axis xyz="0 0 1"/>
         </joint>
-        <transmission name="${name}_steer_transmission">
-            <type>transmission_interface/SimpleTransmission</type>
-            <actuator name="$${name}_steer_motor">
-                <mechanicalReduction>1</mechanicalReduction>
-            </actuator>
-            <joint name="joint_${name}_base_to_${name}_steer">
-                <hardwareInterface>hardware_interface/PositionJointInterface</hardwareInterface>
-            </joint>
-        </transmission>
+        <!--
+            <transmission name="${name}_steer_transmission">
+                <type>transmission_interface/SimpleTransmission</type>
+                <actuator name="$${name}_steer_motor">
+                    <mechanicalReduction>1</mechanicalReduction>
+                </actuator>
+                <joint name="joint_${name}_base_to_${name}_steer">
+                    <hardwareInterface>hardware_interface/PositionJointInterface</hardwareInterface>
+                </joint>
+            </transmission>
+        -->
         <gazebo reference="${name}_steer">
             <material>Gazebo/Blue</material>
@@ -114,17 +116,18 @@
             <mu2>0.5</mu2>
         </gazebo>
-    </xacro:macro>
-    <xacro:macro name="wheel_joint" params="parent child xyz">
+        <gazebo>
+            <plugin name="${name}" filename="libwheel.so">
+                <steer_joint name="joint_${name}_base_to_${name}_steer"/>
+                <drive_joint name="joint_${name}_steer_to_${name}_tire"/>
+            </plugin>
+        </gazebo>
     </xacro:macro>
     <xacro:link_box name="base_link" mass="${body_mass}" length="1" width="1" height="1"/>
-    <xacro:wheel name="wheel_fl" parent="base_link" mass="${wheel_mass}" radius="${wheel_radius}" length="${wheel_length}" xyz="0.2 1 0"/>
-    <xacro:wheel name="wheel_rl" parent="base_link" mass="${wheel_mass}" radius="${wheel_radius}" length="${wheel_length}" xyz="-3 1 0"/>
-    <xacro:wheel name="wheel_rr" parent="base_link" mass="${wheel_mass}" radius="${wheel_radius}" length="${wheel_length}" xyz="-3 -1 0"/>
-    <xacro:wheel name="wheel_fr" parent="base_link" mass="${wheel_mass}" radius="${wheel_radius}" length="${wheel_length}" xyz="0.2 -1 0"/>
+    <xacro:wheel_macro name="wheel_fl" parent="base_link" mass="${wheel_mass}" radius="${wheel_radius}" length="${wheel_length}" xyz="0.2 1 0"/>
+    <xacro:wheel_macro name="wheel_rl" parent="base_link" mass="${wheel_mass}" radius="${wheel_radius}" length="${wheel_length}" xyz="-3 1 0"/>
+    <xacro:wheel_macro name="wheel_rr" parent="base_link" mass="${wheel_mass}" radius="${wheel_radius}" length="${wheel_length}" xyz="-3 -1 0"/>
+    <xacro:wheel_macro name="wheel_fr" parent="base_link" mass="${wheel_mass}" radius="${wheel_radius}" length="${wheel_length}" xyz="0.2 -1 0"/>
     <gazebo>
-        <plugin name="simple_car" filename="libsimple_car.so">
-            <ros>
-                <namespace>/vehicle_namespace</namespace>
-            </ros>
+        <plugin name="vehicle" filename="libvehicle_body.so">
         </plugin>
     </gazebo>

Commit message: implement load transfer equations

File: ws/src/simulator/models/simple_car/model.urdf.xacro (robot description, xacro)
@@ -84,4 +84,8 @@
             <child link="${name}_base"/>
             <axis xyz="0 0 1"/>
+            <!--
+            <dynamics damping="1000" friction="1000"/>
+            <limit lower="-0.15" upper="0.15" effort="1" velocity="0.01"/>
+            -->
         </joint>
         <joint name="joint_${name}_base_to_${name}_steer" type="continuous">

Commit message: refactor mode transition, fix modes in vehicle controller

File: ws/src/simulator/models/simple_car/model.urdf.xacro (robot description, xacro)
@@ -79,13 +79,11 @@
             </collision>
         </link>
-        <joint name="joint_${parent}_to_${name}_base" type="fixed">
+        <joint name="joint_${parent}_to_${name}_base" type="prismatic">
             <origin xyz="${xyz}" rpy="0 0 0"/>
             <parent link="${parent}"/>
             <child link="${name}_base"/>
             <axis xyz="0 0 1"/>
-            <!--
-            <dynamics damping="1000" friction="1000"/>
             <limit lower="-0.15" upper="0.15" effort="1" velocity="0.01"/>
-            -->
+            <safety_controller k_position="100" k_velocity="1"/>
         </joint>
         <joint name="joint_${name}_base_to_${name}_steer" type="continuous">
@@ -117,6 +115,6 @@
         <gazebo reference="${name}_tire">
             <material>Gazebo/Orange</material>
-            <mu1>0.8</mu1>
-            <mu2>0.5</mu2>
+            <mu1>0.9</mu1>
+            <mu2>0.8</mu2>
         </gazebo>
         <gazebo>
@@ -128,8 +126,8 @@
     </xacro:macro>
     <xacro:link_box name="base_link" mass="${body_mass}" length="1" width="1" height="1"/>
-    <xacro:wheel_macro name="wheel_fl" parent="base_link" mass="${wheel_mass}" radius="${wheel_radius}" length="${wheel_length}" xyz="0.2 1 0"/>
-    <xacro:wheel_macro name="wheel_rl" parent="base_link" mass="${wheel_mass}" radius="${wheel_radius}" length="${wheel_length}" xyz="-3 1 0"/>
-    <xacro:wheel_macro name="wheel_rr" parent="base_link" mass="${wheel_mass}" radius="${wheel_radius}" length="${wheel_length}" xyz="-3 -1 0"/>
-    <xacro:wheel_macro name="wheel_fr" parent="base_link" mass="${wheel_mass}" radius="${wheel_radius}" length="${wheel_length}" xyz="0.2 -1 0"/>
+    <xacro:wheel_macro name="wheel_fl" parent="base_link" mass="${wheel_mass}" radius="${wheel_radius}" length="${wheel_length}" xyz="0.2 1.2 0"/>
+    <xacro:wheel_macro name="wheel_rl" parent="base_link" mass="${wheel_mass}" radius="${wheel_radius}" length="${wheel_length}" xyz="-3 1.2 0"/>
+    <xacro:wheel_macro name="wheel_rr" parent="base_link" mass="${wheel_mass}" radius="${wheel_radius}" length="${wheel_length}" xyz="-3 -1.2 0"/>
+    <xacro:wheel_macro name="wheel_fr" parent="base_link" mass="${wheel_mass}" radius="${wheel_radius}" length="${wheel_length}" xyz="0.2 -1.2 0"/>
     <gazebo>
         <plugin name="vehicle" filename="libvehicle_body.so">

Commit message: add experiment folder

File: ws/src/simulator/models/simple_car/model.urdf.xacro (robot description, xacro)
@@ -79,11 +79,11 @@
             </collision>
         </link>
-        <joint name="joint_${parent}_to_${name}_base" type="prismatic">
+        <joint name="joint_${parent}_to_${name}_base" type="fixed">
             <origin xyz="${xyz}" rpy="0 0 0"/>
             <parent link="${parent}"/>
             <child link="${name}_base"/>
             <axis xyz="0 0 1"/>
-            <limit lower="-0.15" upper="0.15" effort="1" velocity="0.01"/>
-            <safety_controller k_position="100" k_velocity="1"/>
+            <limit lower="-1" upper="1" effort="10000000000000000" velocity="100"/>
+            <safety_controller soft_lower_limit="0" soft_upper_limit="0" k_position="1" k_velocity="1"/>
         </joint>
         <joint name="joint_${name}_base_to_${name}_steer" type="continuous">
@@ -117,4 +117,8 @@
             <mu1>0.9</mu1>
             <mu2>0.8</mu2>
+                <!--
+            <mu1>0.0</mu1>
+            <mu2>0.0</mu2>
+                -->
         </gazebo>
         <gazebo>

Commit message: add 3d model for tires

File: ws/src/simulator/models/simple_car/model.urdf.xacro (robot description, xacro)
@@ -69,5 +69,8 @@
                 <origin xyz="0 0 0" rpy="0 0 0"/>
                 <geometry>
+<!--
                     <cylinder radius="${radius}" length="${length}"/>
+-->
+                    <mesh filename="model://simple_car/resources/tire/tire.dae"/>
                 </geometry>
             </visual>
@@ -113,13 +116,11 @@
             <material>Gazebo/Blue</material>
         </gazebo>
+        <!--
         <gazebo reference="${name}_tire">
             <material>Gazebo/Orange</material>
             <mu1>0.9</mu1>
             <mu2>0.8</mu2>
-                <!--
-            <mu1>0.0</mu1>
-            <mu2>0.0</mu2>
-                -->
         </gazebo>
+        -->
         <gazebo>
             <plugin name="${name}" filename="libwheel.so">

Commit message: add tool to simulation

File: ws/src/simulator/models/simple_car/model.urdf.xacro (robot description, xacro)
@@ -18,4 +18,27 @@
                 <geometry>
                     <box size="${length} ${width} ${height}"/>
+                </geometry>
+            </visual>
+            <collision>
+                <origin xyz="0 0 0" rpy="0 0 0"/>
+                <geometry>
+                    <box size="${length} ${width} ${height}"/>
+                </geometry>
+            </collision>
+        </link>
+    </xacro:macro>
+    <xacro:macro name="link_box_mesh" params="name mass length width height mesh_uri">
+        <link name="${name}">
+            <inertial>
+                <origin xyz="0 0 0" rpy="0 0 0"/>
+                <mass value="${mass}"/>
+                <inertia ixx="${1/12*mass*(height**2 + width**2)}" ixy="0" ixz="0"
+                    iyy="${1/12*mass*(height**2 + length**2)}" iyz="0"
+                    izz="${1/12*mass*(length**2 + width**2)}"/>
+            </inertial>
+            <visual>
+                <origin xyz="0 0 0" rpy="0 0 0"/>
+                <geometry>
+                    <mesh filename="${mesh_uri}"/>
                 </geometry>
             </visual>
@@ -131,8 +154,36 @@
     </xacro:macro>
     <xacro:link_box name="base_link" mass="${body_mass}" length="1" width="1" height="1"/>
-    <xacro:wheel_macro name="wheel_fl" parent="base_link" mass="${wheel_mass}" radius="${wheel_radius}" length="${wheel_length}" xyz="0.2 1.2 0"/>
-    <xacro:wheel_macro name="wheel_rl" parent="base_link" mass="${wheel_mass}" radius="${wheel_radius}" length="${wheel_length}" xyz="-3 1.2 0"/>
-    <xacro:wheel_macro name="wheel_rr" parent="base_link" mass="${wheel_mass}" radius="${wheel_radius}" length="${wheel_length}" xyz="-3 -1.2 0"/>
-    <xacro:wheel_macro name="wheel_fr" parent="base_link" mass="${wheel_mass}" radius="${wheel_radius}" length="${wheel_length}" xyz="0.2 -1.2 0"/>
+    <xacro:wheel_macro name="wheel_fl" parent="base_link" mass="${wheel_mass}" radius="${wheel_radius}" length="${wheel_length}" xyz="0.2 1 0"/>
+    <xacro:wheel_macro name="wheel_rl" parent="base_link" mass="${wheel_mass}" radius="${wheel_radius}" length="${wheel_length}" xyz="-3 1 0"/>
+    <xacro:wheel_macro name="wheel_rr" parent="base_link" mass="${wheel_mass}" radius="${wheel_radius}" length="${wheel_length}" xyz="-3 -1 0"/>
+    <xacro:wheel_macro name="wheel_fr" parent="base_link" mass="${wheel_mass}" radius="${wheel_radius}" length="${wheel_length}" xyz="0.2 -1 0"/>
+    <xacro:property name="tool_mass" value="400"/>
+    <link name="tool_link">
+        <inertial>
+            <origin xyz="0 0 0" rpy="0 0 0"/>
+            <mass value="${tool_mass}"/>
+            <inertia ixx="${1/12*tool_mass*(1**2 + 4.5**2)}" ixy="0" ixz="0"
+                iyy="${1/12*tool_mass*(1**2 + 0.5**2)}" iyz="0"
+                izz="${1/12*tool_mass*(0.5**2 + 4.5**2)}"/>
+        </inertial>
+        <visual>
+            <origin xyz="0 0 -0.4" rpy="0 0 1.57"/>
+            <geometry>
+                <mesh filename="model://simple_car/resources/tool/tool.dae"/>
+            </geometry>
+        </visual>
+        <collision>
+            <origin xyz="0 0 0" rpy="0 0 0"/>
+            <geometry>
+                <box size="0.7 5.5 1.2"/>
+            </geometry>
+        </collision>
+    </link>
+    <joint name="joint_tool_to_base_base" type="fixed">
+        <origin xyz="-0.9 0 -0.2" rpy="0 0 0"/>
+        <parent link="base_link"/>
+        <child link="tool_link"/>
+        <axis xyz="0 0 1"/>
+    </joint>
     <gazebo>
         <plugin name="vehicle" filename="libvehicle_body.so">

Commit message: fix (yaw,course) controller, tune yaw controller

File: ws/src/simulator/models/simple_car/model.urdf.xacro (robot description, xacro)
@@ -83,5 +83,5 @@
         <link name="${name}_tire">
             <inertial>
-                <origin xyz="0 0 0" rpy="0 0 0"/>
+                <origin xyz="0 0 0" rpy="${-pi/2} 0 0"/>
                 <mass value="${mass}"/>
                 <inertia ixx="${1/12*mass*(3*radius**2 + length**2)}" ixy="0" ixz="0"
@@ -90,5 +90,5 @@
             </inertial>
             <visual>
-                <origin xyz="0 0 0" rpy="0 0 0"/>
+                <origin xyz="0 0 0" rpy="${-pi/2} 0 0"/>
                 <geometry>
 <!--
@@ -99,5 +99,5 @@
             </visual>
             <collision>
-                <origin xyz="0 0 0" rpy="0 0 0"/>
+                <origin xyz="0 0 0" rpy="${-pi/2} 0 0"/>
                 <geometry>
                     <cylinder radius="${radius}" length="${length}"/>
@@ -110,6 +110,8 @@
             <child link="${name}_base"/>
             <axis xyz="0 0 1"/>
+                <!--
             <limit lower="-1" upper="1" effort="10000000000000000" velocity="100"/>
             <safety_controller soft_lower_limit="0" soft_upper_limit="0" k_position="1" k_velocity="1"/>
+                -->
         </joint>
         <joint name="joint_${name}_base_to_${name}_steer" type="continuous">
@@ -120,8 +122,9 @@
         </joint>
         <joint name="joint_${name}_steer_to_${name}_tire" type="continuous">
-            <origin xyz="0 0 ${-radius - 0.15}" rpy="${-pi/2} 0 0"/>
+            <origin xyz="0 0 ${-radius - 0.15}" rpy="0 0 0"/>
+            <!-- <origin xyz="0 0 ${-radius - 0.15}" rpy="${-pi/2} 0 0"/> -->
             <parent link="${name}_steer"/>
             <child link="${name}_tire"/>
-            <axis xyz="0 0 1"/>
+            <axis xyz="0 1 0"/>
         </joint>
         <!--
@@ -139,11 +142,11 @@
             <material>Gazebo/Blue</material>
         </gazebo>
-        <!--
         <gazebo reference="${name}_tire">
-            <material>Gazebo/Orange</material>
-            <mu1>0.9</mu1>
-            <mu2>0.8</mu2>
+            <!-- <material>Gazebo/Orange</material> -->
+            <!--
+            <mu1>0.3</mu1>
+            <mu2>0.1</mu2>
+            -->
         </gazebo>
-        -->
         <gazebo>
             <plugin name="${name}" filename="libwheel.so">
@@ -158,4 +161,5 @@
     <xacro:wheel_macro name="wheel_rr" parent="base_link" mass="${wheel_mass}" radius="${wheel_radius}" length="${wheel_length}" xyz="-3 -1 0"/>
     <xacro:wheel_macro name="wheel_fr" parent="base_link" mass="${wheel_mass}" radius="${wheel_radius}" length="${wheel_length}" xyz="0.2 -1 0"/>
+    <!--
     <xacro:property name="tool_mass" value="400"/>
     <link name="tool_link">
@@ -186,4 +190,5 @@
         <axis xyz="0 0 1"/>
     </joint>
+    -->
     <gazebo>
         <plugin name="vehicle" filename="libvehicle_body.so">

Commit message: make a few plots

File: ws/src/simulator/models/simple_car/model.urdf.xacro (robot description, xacro)
@@ -10,7 +10,5 @@
                 <origin xyz="0 0 0" rpy="0 0 0"/>
                 <mass value="${mass}"/>
-                <inertia ixx="${1/12*mass*(height**2 + width**2)}" ixy="0" ixz="0"
-                    iyy="${1/12*mass*(height**2 + length**2)}" iyz="0"
-                    izz="${1/12*mass*(length**2 + width**2)}"/>
+                <inertia ixx="${1/12*mass*(height**2 + width**2)}" ixy="0" ixz="0" iyy="${1/12*mass*(height**2 + length**2)}" iyz="0" izz="${1/12*mass*(length**2 + width**2)}"/>
             </inertial>
             <visual>
@@ -33,7 +31,5 @@
                 <origin xyz="0 0 0" rpy="0 0 0"/>
                 <mass value="${mass}"/>
-                <inertia ixx="${1/12*mass*(height**2 + width**2)}" ixy="0" ixz="0"
-                    iyy="${1/12*mass*(height**2 + length**2)}" iyz="0"
-                    izz="${1/12*mass*(length**2 + width**2)}"/>
+                <inertia ixx="${1/12*mass*(height**2 + width**2)}" ixy="0" ixz="0" iyy="${1/12*mass*(height**2 + length**2)}" iyz="0" izz="${1/12*mass*(length**2 + width**2)}"/>
             </inertial>
             <visual>
@@ -56,7 +52,5 @@
                 <origin xyz="0 0 0" rpy="0 0 0"/>
                 <mass value="1"/>
-                <inertia ixx="1" ixy="0" ixz="0"
-                    iyy="1" iyz="0"
-                    izz="1"/>
+                <inertia ixx="1" ixy="0" ixz="0" iyy="1" iyz="0" izz="1"/>
             </inertial>
             <visual>
@@ -70,7 +64,5 @@
             <inertial>
                 <mass value="1"/>
-                <inertia ixx="1" ixy="0" ixz="0"
-                    iyy="1" iyz="0"
-                    izz="1"/>
+                <inertia ixx="1" ixy="0" ixz="0" iyy="1" iyz="0" izz="1"/>
             </inertial>
             <visual>
@@ -85,12 +77,10 @@
                 <origin xyz="0 0 0" rpy="${-pi/2} 0 0"/>
                 <mass value="${mass}"/>
-                <inertia ixx="${1/12*mass*(3*radius**2 + length**2)}" ixy="0" ixz="0"
-                    iyy="${1/12*mass*(3*radius**2 + length**2)}" iyz="0"
-                    izz="${1/2*mass*radius**2}"/>
+                <inertia ixx="${1/12*mass*(3*radius**2 + length**2)}" ixy="0" ixz="0" iyy="${1/12*mass*(3*radius**2 + length**2)}" iyz="0" izz="${1/2*mass*radius**2}"/>
             </inertial>
             <visual>
                 <origin xyz="0 0 0" rpy="${-pi/2} 0 0"/>
                 <geometry>
-<!--
+                    <!--
                     <cylinder radius="${radius}" length="${length}"/>
 -->
@@ -110,5 +100,5 @@
             <child link="${name}_base"/>
             <axis xyz="0 0 1"/>
-                <!--
+            <!--
             <limit lower="-1" upper="1" effort="10000000000000000" velocity="100"/>
             <safety_controller soft_lower_limit="0" soft_upper_limit="0" k_position="1" k_velocity="1"/>
@@ -166,7 +156,5 @@
             <origin xyz="0 0 0" rpy="0 0 0"/>
             <mass value="${tool_mass}"/>
-            <inertia ixx="${1/12*tool_mass*(1**2 + 4.5**2)}" ixy="0" ixz="0"
-                iyy="${1/12*tool_mass*(1**2 + 0.5**2)}" iyz="0"
-                izz="${1/12*tool_mass*(0.5**2 + 4.5**2)}"/>
+            <inertia ixx="${1/12*tool_mass*(1**2 + 4.5**2)}" ixy="0" ixz="0" iyy="${1/12*tool_mass*(1**2 + 0.5**2)}" iyz="0" izz="${1/12*tool_mass*(0.5**2 + 4.5**2)}"/>
         </inertial>
         <visual>
